Commit message: Complete step 2: add camera and publish tf data

File: urdf/pointcloud_camera.xacro (robot description, xacro)
@@ -1,7 +1,16 @@
 <?xml version="1.0"?>
 <robot xmlns:xacro="http://www.ros.org/wiki/xacro" name="gurdy">
+    <!--
+    /home/user/simulation_ws/src/robotnik_sensors_master_project/robotnik_sensors/urdf/all_sensors.urdf.xacro
+    /home/user/simulation_ws/src/robotnik_sensors_master_project/robotnik_sensors/urdf/intel_r430.urdf.xacro
+    -->
+    <xacro:include filename="$(find robotnik_sensors)/urdf/all_sensors.urdf.xacro"/>
     <xacro:property name="pc_cam_body_link_radius" value="0.1"/>
     <xacro:property name="pc_cam_body_link_length" value="0.05"/>
     <xacro:property name="pc_cam_body_link_mass" value="50"/>
+    <!-- Camera at a distance of 1.2 meters in the z axis with respect from the pc_cam_base_link.
+         The camera has an inclination of 30º in the pitch axis.-->
+    <xacro:property name="camera_height_from_base" value="1.2"/>
+    <xacro:property name="camera_pitch" value="1.047"/>
     <!-- The same for all objects-->
     <xacro:property name="kp" value="1000.0"/>
@@ -37,14 +46,35 @@
             </visual>
         </link>
+        <!--
+        <xacro:macro name="sensor_r430" params="prefix parent prefix_topic:='front_rgbd_camera' *origin">
+            <joint name="${prefix}_camera_joint" type="fixed">
+                <xacro:insert_block name="origin" />
+                <parent link="${parent}"/>
+                <child link="${prefix}_camera_link" />
+            </joint>
+            ...
+        -->
+        <xacro:sensor_r430 prefix="pc_cam" parent="pc_cam_body_link" >
+            <origin xyz="0 0 ${camera_height_from_base}" rpy="0 0 ${camera_pitch}"/>
+        </xacro:sensor_r430>
         <gazebo reference="pc_cam_body_link">
+            <!--
             <kp>${kp}</kp>
             <kd>${kd}</kd>
             <mu1>${mu1}</mu1>
             <mu2>${mu2}</mu2>
+            -->
         </gazebo>
-        <joint name="fixed" type="fixed">
+        <joint name="base_joint" type="fixed">
             <parent link="base_link"/>
             <child link="pc_cam_body_link"/>
         </joint>
+        <!--
+        <joint name="pc_cam_body_front_rgbd_camera_link" type="fixed">
+            <parent link="base_link"/>
+            <child link="pc_cam_body_link"/>
+            <origin xyz="0 0 ${camera_height_from_base}" rpy="0 0 ${camera_pitch}"/>
+        </joint>
+        -->
     </xacro:macro>
     <xacro:pc_cam/>

Commit message: Camera base is zinc yellow in both rviz and gazebo

File: urdf/pointcloud_camera.xacro (robot description, xacro)
@@ -23,4 +23,8 @@
                 izz="${mass*(r*r)/2}" />
     </xacro:macro >
+    <!-- For RVIZ -->
+    <material name="zinc_yellow">
+        <color rgba="0.9804 0.7922 0.1882 1"/>
+    </material>
     <!-- The support base for the camera -->
     <xacro:macro name="pc_cam">
@@ -44,7 +48,9 @@
                     <cylinder radius="${pc_cam_body_link_radius}" length="${pc_cam_body_link_length}"/>
                 </geometry>
+                <material name="zinc_yellow"/>
             </visual>
         </link>
         <!--
+        From the camera's XACRO:
         <xacro:macro name="sensor_r430" params="prefix parent prefix_topic:='front_rgbd_camera' *origin">
             <joint name="${prefix}_camera_joint" type="fixed">
@@ -59,10 +65,5 @@
         </xacro:sensor_r430>
         <gazebo reference="pc_cam_body_link">
-            <!--
-            <kp>${kp}</kp>
-            <kd>${kd}</kd>
-            <mu1>${mu1}</mu1>
-            <mu2>${mu2}</mu2>
-            -->
+            <material>Gazebo/ZincYellow</material>
         </gazebo>
         <joint name="base_joint" type="fixed">
@@ -70,11 +71,4 @@
             <child link="pc_cam_body_link"/>
         </joint>
-        <!--
-        <joint name="pc_cam_body_front_rgbd_camera_link" type="fixed">
-            <parent link="base_link"/>
-            <child link="pc_cam_body_link"/>
-            <origin xyz="0 0 ${camera_height_from_base}" rpy="0 0 ${camera_pitch}"/>
-        </joint>
-        -->
     </xacro:macro>
     <xacro:pc_cam/>

Commit message: Rename camera launch file Bug fix: robot state publisher name conflict Bug fix: base_link name conflict New RVIZ config for Part 4: TF

File: urdf/pointcloud_camera.xacro (robot description, xacro)
@@ -29,5 +29,5 @@
     <!-- The support base for the camera -->
     <xacro:macro name="pc_cam">
-        <link name="base_link">
+        <link name="pc_cam_base_link">
         </link>
         <link name="pc_cam_body_link">
@@ -68,5 +68,5 @@
         </gazebo>
         <joint name="base_joint" type="fixed">
-            <parent link="base_link"/>
+            <parent link="pc_cam_base_link"/>
             <child link="pc_cam_body_link"/>
         </joint>

Commit message: Fix camera position Fix static transform launch file Add currently unused python files that do the static transform as well

File: urdf/pointcloud_camera.xacro (robot description, xacro)
@@ -12,5 +12,5 @@
          The camera has an inclination of 30º in the pitch axis.-->
     <xacro:property name="camera_height_from_base" value="1.2"/>
-    <xacro:property name="camera_pitch" value="1.047"/>
+    <xacro:property name="camera_pitch" value="0.52"/>
     <!-- The same for all objects-->
     <xacro:property name="kp" value="1000.0"/>
@@ -62,5 +62,5 @@
         -->
         <xacro:sensor_r430 prefix="pc_cam" parent="pc_cam_body_link" >
-            <origin xyz="0 0 ${camera_height_from_base}" rpy="0 0 ${camera_pitch}"/>
+            <origin xyz="0 0 ${camera_height_from_base}" rpy="0 ${camera_pitch} 0"/>
         </xacro:sensor_r430>
         <gazebo reference="pc_cam_body_link">
